File: MainBoard/MainBoard/MainBoard.kicad_pcb (KiCad board)
At the start: 6 copper layers, 45 x 45.6 mm, 41 parts, among them IC1 BQ25171QWDRCRQ1, J1 KH-TYPE-C-16P, U1 STM32L496VGY6PTR, U2 MX25R1635FZUIL0, U3 SI3477DV-T1-GE3, U4 SI3477DV-T1-GE3, U5 TPS63802DLAR, U6 FUSB302BMPX

Commit message: Schematic work
Parts:
- added C21: 1uF, Capacitor_SMD:C_0402_1005Metric_Pad0.74x0.62mm_HandSolder, F.Cu at (90.0, 76.5)
- added C22: 100nF, Capacitor_SMD:C_0402_1005Metric_Pad0.74x0.62mm_HandSolder, F.Cu at (90.0, 78.5)
- added C23: 470pF, Capacitor_SMD:C_0402_1005Metric_Pad0.74x0.62mm_HandSolder, F.Cu at (90.0, 80.4)
- added C24: 470pF, Capacitor_SMD:C_0402_1005Metric_Pad0.74x0.62mm_HandSolder, F.Cu at (90.0, 82.4)
- added R8: 4.7k, Resistor_SMD:R_0402_1005Metric_Pad0.72x0.64mm_HandSolder, F.Cu at (84.6, 79.8)
- added R9: 4.7k, Resistor_SMD:R_0402_1005Metric_Pad0.72x0.64mm_HandSolder, F.Cu at (84.6, 81.8)
Connections:
- C19 pad 1: Net-(U5-VOUT) -> +3.3V
- C20 pad 1: Net-(U5-VOUT) -> +3.3V
- J1 pad A5: unconnected-(J1-CC1-PadA5) -> Net-(J1-CC1)
- J1 pad B5: unconnected-(J1-CC2-PadB5) -> Net-(J1-CC2)
- R6 pad 1: Net-(U5-VOUT) -> +3.3V
- U5 pad 6: Net-(U5-VOUT) -> +3.3V
- U6 pad 11: unconnected-(U6-CC1-Pad11) -> Net-(J1-CC1)
- U6 pad 14: unconnected-(U6-CC2-Pad14) -> Net-(J1-CC2)
- U6 pad 15: unconnected-(U6-EPAD-Pad15) -> GND
- U6 pad 2: unconnected-(U6-VBUS-Pad2) -> Net-(D1-A)
- U6 pad 3: unconnected-(U6-VDD-Pad3) -> +3.3V
- U6 pad 4: unconnected-(U6-VDD-Pad4) -> +3.3V
- U6 pad 6: unconnected-(U6-SCL-Pad6) -> I2C1_SCL
- U6 pad 7: unconnected-(U6-SDA-Pad7) -> I2C1_SDA
- U6 pad 8: unconnected-(U6-GND-Pad8) -> GND
- U6 pad 9: unconnected-(U6-GND-Pad9) -> GND

Commit message: Schematic Work
Parts:
- added MOD1: RFM98W-433S2, inspirefly:XCVR_RFM98W-433S2, F.Cu at (85.6, 76.4)
- moved C10 47.8 mm to (120.6, 48.5)
- moved C11 47.8 mm to (120.6, 50.5)
- moved C12 47.8 mm to (120.6, 52.5)
- moved C23 47.8 mm to (131.1, 55.9)
- moved C24 47.8 mm to (131.1, 57.9)
- moved C21 47.8 mm to (131.1, 52.0)
- moved C22 47.8 mm to (131.1, 54.0)
- moved C7 47.8 mm to (120.6, 42.6)
- moved C8 47.8 mm to (120.6, 44.6)
- moved C9 47.8 mm to (120.6, 46.6)
- moved C18 47.8 mm to (131.0, 45.7)
- moved C4 47.8 mm to (117.4, 48.5)
- moved C5 47.8 mm to (117.4, 50.5)
- moved C6 47.8 mm to (117.4, 52.5)
- moved R2 47.8 mm to (140.1, 46.8)
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
Commit message: Schematic work
Parts:
- added C25: 100nF, Capacitor_SMD:C_0402_1005Metric_Pad0.74x0.62mm_HandSolder, F.Cu at (130.8, 64.7)
- added C26: 100nF, Capacitor_SMD:C_0402_1005Metric_Pad0.74x0.62mm_HandSolder, F.Cu at (130.8, 66.7)
- added C27: 100nF, Capacitor_SMD:C_0402_1005Metric_Pad0.74x0.62mm_HandSolder, F.Cu at (130.8, 68.7)
- added C28: 22pF, Capacitor_SMD:C_0402_1005Metric_Pad0.74x0.62mm_HandSolder, F.Cu at (130.8, 70.6)
- added C29: 22pF, Capacitor_SMD:C_0402_1005Metric_Pad0.74x0.62mm_HandSolder, F.Cu at (130.8, 72.6)
- added R10: 10k, Resistor_SMD:R_0402_1005Metric_Pad0.72x0.64mm_HandSolder, F.Cu at (130.9, 62.7)
- added U7: BNO086, inspirefly:BNO086, F.Cu at (100.8, 73.5)
- added Y1: 9HT11-32.768KBZF-T, Crystal:Crystal_SMD_2012-2Pin_2.0x1.2mm_HandSoldering, F.Cu at (106.2, 72.4)
- moved U4 2.51 mm to (107.2, 81.0)
Connections:
- IC1 pad 3: unconnected-(IC1-~{CE}-Pad3) -> CHARGE_DISABLE
