File: MainBoard/MainBoard.kicad_sch (KiCad schematic)
At the start: 93 parts, among them J1 KH-TYPE-C-16P, Q1 PMV19XNEAR, Q2 PMV19XNEAR, Q3 PMV19XNEAR, Q4 PMV19XNEAR, U2 SI3477DV-T1-GE3, U3 STM32L496VGY6PTR, U4 FUSB302BMPX, U5 BNO086, U6 TPS63802DLAR, U7 SI3477DV-T1-GE3, U8 BQ25756ERRVR, U9 TCAN332DCNR, Y1 9HT11-32.768KBZF-T

Commit message: Adding cutoff circuits and others
Added 3.3V and Bat Voltage current sense and cutoff cirucits

Also changed footprints to non-hand solder for 0402

And changed I2C pullups to an array
Parts:
- removed R1, R2, R3, R4, R5, R6, R7, R9: 2.2k, Resistor_SMD:R_0402_1005Metric_Pad0.72x0.64mm_HandSolder, symbol Device:R_US
- added C28, C3: 100nF, Capacitor_SMD:C_0402_1005Metric, symbol Device:C
- added R31, R33: 5m, Resistor_SMD:R_1206_3216Metric_Pad1.30x1.75mm_HandSolder, symbol Device:R_US
- added R32, R34: 100K, Resistor_SMD:R_0402_1005Metric, symbol Device:R_US
- added RN1: YC158TJR-072K2L, inspirefly:RESCAXE64P320X160X70-10N, symbol inspirefly:YC158TJR-072K2L
- added U1, U11: INA185A4IDRLR, inspirefly:SOT_INA185_TEX, symbol inspirefly:INA185A1IDRLR
- added U10, U12: SI3477DV-T1-GE3, inspirefly:SOT_V-T1-GE3_VIS-M, symbol inspirefly:SI3477DV-T1-GE3
- C1, C10, C11, C12, C13, C14, C15, C16, C17, C18, C19, C2, C20, C21, C22, C23, C24, C25, C26, C27, C30, C31, C32, C33, C36, C37, C38, C4, C41, C42, C43, C44, C45, C5, C6, C7, C8, C9: footprint Capacitor_SMD:C_0402_1005Metric_Pad0.74x0.62mm_HandSolder -> Capacitor_SMD:C_0402_1005Metric
- C34, C35: footprint Capacitor_SMD:C_1206_3216Metric_Pad1.33x1.80mm_HandSolder -> Capacitor_SMD:C_0402_1005Metric
- R10, R11, R12, R13, R14, R15, R16, R17, R18, R19, R20, R22, R23, R24, R25, R26, R27, R28, R30, R8: footprint Resistor_SMD:R_0402_1005Metric_Pad0.72x0.64mm_HandSolder -> Resistor_SMD:R_0402_1005Metric
- R21: footprint Resistor_SMD:R_1206_3216Metric_Pad1.30x1.75mm_HandSolder -> Resistor_SMD:R_0402_1005Metric
Connections:
- net +3.3V: now also C28.2, C3.2, R31.1, RN1.10, RN1.5, U1.3 (IN+), U1.6 (VS), U11.6 (VS)
- net BAT+: now also R33.1, U11.3 (IN+)
- net GND: now also C28.1, C3.1, U1.2 (GND), U1.5 (REF), U11.2 (GND), U11.5 (REF)
- net I2C1_SCL: now also RN1.2
- net I2C1_SDA: now also RN1.1
- net I2C2_SCL: now also RN1.4
- net I2C2_SDA: now also RN1.3
- net I2C3_SCL: now also RN1.8
- net I2C3_SDA: now also RN1.9
- new net: R31.2, R32.1, U1.4 (IN-), U10.4 (S)
- new net: R33.2, R34.1, U11.4 (IN-), U12.4 (S)
- new net ADC1_A1: U1.1 (OUT)
- new net ADC1_A2: U11.1 (OUT)
- new net BOARD_OUT_3.3V: U10.1 (D), U10.2 (D), U10.5 (D), U10.6 (D)
- new net BOARD_OUT_BAT: U12.1 (D), U12.2 (D), U12.5 (D), U12.6 (D)
- new net EXTERNAL_3.3V_CUTOFF: R32.2, U10.3 (G)
- new net EXTERNAL_BAT_CUTOFF: R34.2, U12.3 (G)
- new net I2C4_SCL: RN1.6
- new net I2C4_SDA: RN1.7
Other:
- note added: "3.3/ 2^16 = 50.35uV per LSB"
- note added: "4.2/ 2^16 = 64.087uV per LSB"
- note added: "50.35uV / (200 x .005) = 50.35uA per LSB"
- note added: "64.087uV / (200 x .005) = 64.087uA per LSB"
- note added: "External board cutoff + current sense (3.3V)"
- note added: "External board cutoff + current sense (Battery Voltage)"
- note added: "Note that this equation will change based on battery voltage"
- note added: "With 16bit oversample-"
- moved on the sheet: U2
