File: MainBoard/MainBoard.kicad_sch (KiCad schematic)
At the start: 110 parts, among them J2 USB4110-GF-A, J3 M55-7104042R, J4 Conn_01x04_Pin, J5 Conn_01x02_Pin, Q1 PMV19XNEAR, Q2 PMV19XNEAR, Q3 PMV19XNEAR, Q4 PMV19XNEAR, SW1 SW_TL1015AF160QG, SW2 SW_TL1015AF160QG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

Commit message: Changes to USB and routing
Added ESD protection IC
Routed USB Differential to STM
Parts:
- added C47: 100nF, Capacitor_SMD:C_0402_1005Metric, symbol Device:C
- added CR1: USBLC6-2SC6, inspirefly:SOT23-6L_STM, symbol inspirefly:USBLC6-2SC6
Connections:
- net GND: now also C47.2, CR1.2
- net USB_D+: now also CR1.4; no longer J2.A6 (DP1), J2.B6 (DP2)
- net USB_D-: now also CR1.6; no longer J2.A7 (DN1), J2.B7 (DN2)
- net at D1.2 (A), J2.A4-B9 (VBUS), J2.A9-B4 (VBUS)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: now also C47.1, CR1.5
- new net: CR1.1, J2.A7 (DN1), J2.B7 (DN2)
- new net: CR1.3, J2.A6 (DP1), J2.B6 (DP2)
Other:
- moved on the sheet: C1, C18, C2, C26, C27, C6, C7, L1, R11, R12, R8, TP3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

Commit message: Added E-Fuse/ battery protection IC
Added and routed new IC for battery

- will have to figure out cutoff but that can be done later imo
Parts:
- removed JP1: Footswitch_Disable, inspirefly:SmallJumper, symbol Jumper:SolderJumper_2_Open
- removed R13: 100K, Resistor_SMD:R_0402_1005Metric, symbol Device:R_US
- removed TP1: BatBeforeCutoff, TestPoint:TestPoint_Pad_D1.0mm, symbol Connector:TestPoint
- removed TP2: Bat+, TestPoint:TestPoint_Pad_D1.0mm, symbol Connector:TestPoint
- removed U7: SI3477DV-T1-GE3, inspirefly:SOT_V-T1-GE3_VIS-M, symbol inspirefly:SI3477DV-T1-GE3
- added C48, C49: 10nF, Capacitor_SMD:C_0402_1005Metric, symbol Device:C
- added C50: 47uF, Capacitor_SMD:C_1206_3216Metric_Pad1.33x1.80mm_HandSolder, symbol Device:C
- added R3: 143k, Resistor_SMD:R_0402_1005Metric, symbol Device:R_US
- added R4: 100k, Resistor_SMD:R_0402_1005Metric, symbol Device:R_US
- added R5: 1k, Resistor_SMD:R_0402_1005Metric, symbol Device:R_US
- added U13: TPS259472ARPWR, inspirefly:RPW0010A-MFG, symbol inspirefly:TPS259470ARPWR
Connections:
- net BAT+: now also BT1.P, BT2.P, R3.2, U13.5 (IN); no longer C18.1, R33.1, R35.2, U11.3 (IN+), U2.4 (S), U6.1 (EN), U6.10 (VIN)
- net GND: now also C48.1, C49.1, C50.2, R4.1, R5.1, U13.8 (GND)
- new net: C48.2, U13.10 (ITIMER)
- new net: R3.1, R4.2, U13.1 (EN_UVLO)
- new net: C49.2, U13.7 (dVdt)
- new net: R5.2, U13.9 (ILM)
- new net PROTECTED_VOLTAGE: C18.1, C50.1, R33.1, R35.2, U11.3 (IN+), U13.6 (OUT), U2.4 (S), U6.1 (EN), U6.10 (VIN)
- no-connect marks 65 -> 68
Other:
- note added: "Overcurrent 3.334A as 3334 / 1k = 3.334A"
- note added: "Undervoltage at 2.916V V_UV = (1.2(143k + 100k)) / 100k"
- moved on the sheet: BT1, BT2, C33, C39, R25, U9

Commit message: Pushing BOM and changes
Had to change one resistor footprint and routing
Parts:
- R15: footprint Resistor_SMD:R_0402_1005Metric -> Resistor_SMD:R_0805_2012Metric
Changed lines of the file:
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@@
 			)
 		)
-		(property "Footprint" "Resistor_SMD:R_0402_1005Metric"
+		(property "Footprint" "Resistor_SMD:R_0805_2012Metric"
 			(at 345.186 226.314 90)
 			(effects

Commit message: Mounting pad additions, footswitch and BOM changes
Parts:
- added H1, H2, H3, H4: MountingHole_Pad, inspirefly:MoutingPad, symbol Mechanical:MountingHole_Pad
- added JP1: FTSW EN, inspirefly:SmallJumper, symbol Jumper:Jumper_2_Open
- R14: value 143k -> 82.5k
- R15: value 250k -> 143k; footprint Resistor_SMD:R_0805_2012Metric -> Resistor_SMD:R_0402_1005Metric
Connections:
- net GND: now also H1.1, H2.1, H3.1, H4.1
- net JTMS/SWDIO: now also J4.4 (Pin_4); no longer J4.1 (Pin_1)
- net NRST: now also J4.1 (Pin_1); no longer J4.4 (Pin_4)
- net at R3.1, R4.2, U13.1 (EN_UVLO): now also JP1.2 (B)
- net FOOTSWITCH: now reaches J3.B13
- net FOOTSWITCH: now also JP1.1 (A)
- net BAT_PULLDOWN: no longer names the net of U3.F3 (PD14)
Other:
- note added: "Footswitch Logic NO: Floating / NC NC: Ground"
- note added: "Overvoltage (pin 2) is left open to have clamp at 5.7V"

Commit message: Final Board Order Changes for Mainboard
Parts:
- added J1: FTSH-107-01-L-DV-K-A, inspirefly:SAMTEC_FTSH-107-01-L-DV-K-A, symbol inspirefly:FTSH-107-01-L-DV-K-A
- added JP2: GND_DETECT, inspirefly:SmallJumper, symbol Jumper:Jumper_2_Open
- added R6: 100k, Resistor_SMD:R_0402_1005Metric, symbol Device:R_US
- added R7: 10k, Resistor_SMD:R_0402_1005Metric, symbol Device:R_US
- added R9: Heater, inspirefly:HeaterConnection, symbol Device:Heater
- added TH1: NRBG104F3435B2F, inspirefly:NRBG104F3435B2F, symbol Device:Thermistor_NTC
- D2: value LED -> LTST-S270KRKT; footprint LED_SMD:LED_0402_1005Metric -> LED_SMD:LED_0603_1608Metric_Pad1.05x0.95mm_HandSolder
Connections:
- net +3.3V: now also J1.03, R7.1
- net ANT_SPI2_SCK: now also U3.D3 (PA9); no longer U3.K3 (PB10)
- net GND: now also J1.05, J1.07, JP2.1 (A), R6.2, R9.2, TH1.2
- net JTCK/SWCLK: now also J1.06
- net JTMS/SWDIO: now also J1.04
- net NRST: now also J1.12, R7.2
- net SWO: now also J1.08
- net THERMISTOR_FEEDBACK: now also TH1.1
- net JTDI: now reaches U3.A2 (PA15)
- net JTDI: now also J1.10
- net DEBUG_LPUART_TX: now reaches U3.J3 (PB11)
- net DEBUG_LPUART_TX: now also J1.13
- net at U2.1 (D): now also U2.2 (D), U2.5 (D), U2.6 (D), R9.1
- new net: J1.11, JP2.2 (B), R6.1
- new net DEBUG_LPUART_RX: J1.14, U3.K3 (PB10)
Other:
- moved on the sheet: J4, J5
