File: BatteryBoard/BatteryBoard.kicad_sch (KiCad schematic)
At the start: 69 parts, among them J1 M55-7102642R, Q1 PMPB13XNE,115, Q2 PMPB13XNE,115, Q3 PMPB13XNE,115, Q5 PMPB13XNE,115, U1 INA185A4IDRLR, U10 SI3477DV-T1-GE3, U13 TPS259472ARPWR, U2 SI3477DV-T1-GE3, U6 TPS63802DLAR, U8 BQ25756ERRVR

Commit message: Flight Controller updates
Connections:
- net BOARD_OUT_3.3V is gone; now on net PAYLOAD_3.3V: U10.1 (D), U10.2 (D), U10.5 (D), U10.6 (D)
- net EXTERNAL_3.3V_CUTOFF is gone; now on net PAYLOAD_3.3V_EN: R32.2, U10.3 (G)
- net +3.3V: now also J1.A8, J1.A9; no longer J1.A11, J1.A12, J1.A13
- net ADC1_A1: now also J1.B10
- net BAT_VOLTAGE: now also J1.A11, J1.A12, J1.A13; no longer J1.B10, J1.B11, J1.B12, J1.B13
- net EXTERNAL_VOLTAGE: no longer J1.A4
- net GND: now also J1.A4; no longer J1.A8, J1.A9

Commit message: Routing and schematic work on most boards
Parts:
- removed C1, C34, C50: 47uF, Capacitor_SMD:C_1206_3216Metric_Pad1.33x1.80mm_HandSolder, symbol Device:C
- removed H1, H2, H3, H4: MountingHole_Pad, inspirefly:MoutingPad, symbol Mechanical:MountingHole_Pad
- added C19, C20, C21, C22, C23, C24, C25: 10uF, Capacitor_SMD:C_0603_1608Metric, symbol Device:C
- added C47, C51, C53, C54, C55, C58: 22uF, Capacitor_SMD:C_1210_3225Metric, symbol Device:C
- added L3: 470nH, Inductor_SMD:L_0805_2012Metric_Pad1.05x1.20mm_HandSolder, symbol Device:L
- added Q4, Q6: T2N7002AK,LM, Package_TO_SOT_SMD:SOT-23-3, symbol Simulation_SPICE:NMOS
- added R13: 280k, Resistor_SMD:R_0402_1005Metric_Pad0.72x0.64mm_HandSolder, symbol Device:R_US
- added R22: 50k, Resistor_SMD:R_0402_1005Metric_Pad0.72x0.64mm_HandSolder, symbol Device:R_US
- added R36, R37: 100, Resistor_SMD:R_0402_1005Metric_Pad0.72x0.64mm_HandSolder, symbol Device:R_US
- added R38: 10k, Resistor_SMD:R_0402_1005Metric_Pad0.72x0.64mm_HandSolder, symbol Device:R_US
- added TH2: NRBG104F3435B2F, inspirefly:NRBG104F3435B2F, symbol Device:Thermistor_NTC
- added U3: TPS2117DRLR, inspirefly:SOTFL50P160X60-8N, symbol inspirefly:TPS2117DRLR
- added U7: TPS63802DLAR, inspirefly:VREG_TPS63802DLAR, symbol inspirefly:TPS63802DLAR
- C18, C36, C37: footprint Capacitor_SMD:C_0402_1005Metric_Pad0.74x0.62mm_HandSolder -> Capacitor_SMD:C_0603_1608Metric
- C35, C39, C40: value 47uF -> 22uF; footprint Capacitor_SMD:C_1206_3216Metric_Pad1.33x1.80mm_HandSolder -> Capacitor_SMD:C_1210_3225Metric
- L1: footprint Inductor_SMD:L_0805_2012Metric_Pad1.15x1.40mm_HandSolder -> Inductor_SMD:L_0805_2012Metric_Pad1.05x1.20mm_HandSolder
- R3: value 143k -> 649k
- R32, R35: value 100k -> 10k
- R4: value 100k -> 348k
- R5: value 1k -> 750
Connections:
- net BAT_VOLTAGE is gone; now on net GND: J1.A11, J1.A12, J1.A13
- net +3.3V: now also J1.B7, J1.B8, J1.B9, C22.1, C24.1, C25.1, U3.2 (VOUT), U3.4 (PR1), U3.5 (MODE), U3.7 (VOUT__1); no longer J1.A10, J1.A8, J1.A9, R11.1, U6.6 (VOUT)
- net ADC1_A1: now also J1.A3; no longer J1.B10
- net BAT+: now also C54.1, C55.1; no longer C39.1
- net BATMANG_INT_DIN: now also J1.A8; no longer J1.B4
- net BAT_HEAT_EN: now also J1.A5, R36.2; no longer J1.B8, R35.1, U2.3 (G)
- net EXTERNAL_VOLTAGE: now also J1.B1, J1.B2, J1.B3, C47.1, C51.1; no longer C40.1, J1.A1, J1.A2, J1.A3
- net FOOTSWITCH: now also J1.A9; no longer J1.B5
- net GND: now also J1.A10, C19.2, C20.2, C21.2, C22.2, C23.1, C24.2, C25.2, C47.2, C51.2, C53.2, C54.2, C55.2, C58.2, Q4.3 (S), Q6.3 (S), R22.2, TH2.2, U3.1 (GND), U7.2 (MODE), U7.3 (AGND), U7.8 (GND); no longer J1.A4, J1.A5, J1.A6, J1.A7
- net I2C2_SCL: now also J1.A6; no longer J1.B7
- net I2C2_SDA: now also J1.A7; no longer J1.B6
- net PAYLOAD_3.3V: now also J1.B4, J1.B5, J1.B6, C23.2; no longer J1.B1, J1.B2, J1.B3
- net PAYLOAD_3.3V_EN: now also J1.A4, R37.2; no longer J1.B9, R32.2, U10.3 (G)
- net PROTECTED_VOLTAGE: now also J1.B10, J1.B11, J1.B12, J1.B13, C20.1, C58.1, U7.1 (EN), U7.10 (VIN)
- net at C35.1, Q5.1, Q5.2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: now also C40.1
- net at Q2.1, Q2.2, Q2.5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: now also C39.1, C53.1
- new net: Q4.1 (D), R35.1, U2.3 (G)
- new net: Q4.2 (G), R36.1
- new net: Q6.1 (D), R32.2, U10.3 (G)
- new net: R13.2, R22.1, U7.4 (FB)
- new net: C21.1, R13.1, U3.6 (VIN2), U7.6 (VOUT)
- new net: L3.2, U7.7 (L2)
- new net: L3.1, U7.9 (L1)
- new net: Q6.2 (G), R37.1
- new net: C19.1, R11.1, U3.3 (VIN1), U6.6 (VOUT)
- new net ADC1_A2: J1.A2, R38.2, TH2.1
- new net EN_THERMISTOR_READ: J1.A1, R38.1
- no-connect marks 6 -> 8
Other:
- note added: "3.3V Regulators with Priority Mux output to 3.3V"
- note added: "Battery Heater Connection + NTC Termistors"
- note added: "Overcurrent 3.334A as 3334 / 750 = 4.45A"
- note added: "Undervoltage at 3.12V V_UV = (1.2(649k + 348k)) / 348k * (1 - .092 hystersis)"
- note removed: "3.3V Regulator"
- note removed: "Battery Heater Connection"
- note removed: "Overcurrent 3.334A as 3334 / 1k = 3.334A"
- note removed: "Undervoltage at 2.916V V_UV = (1.2(143k + 100k)) / 100k"
- moved on the sheet: C18, L1, R11, R12, R35, R9, TH1, TP3, U2, U6

Commit message: Finalize board work + BOM work
Parts:
- L2: footprint inspirefly:IHLP1212BZEZ2R2M1Z -> inspirefly:IND_SRP4020FA-2R2M_BRN
Other:
- note added: "SRP4020FA-2R2M"
- note removed: "IHLP1212BZEZ2R2M1Z"
Changed lines of the file:
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@@
 		)
 	)
-	(text "IHLP1212BZEZ2R2M1Z"
+	(text "SRP4020FA-2R2M"
 		(exclude_from_sim no)
-		(at 426.212 325.882 0)
+		(at 426.974 325.882 0)
 		(effects
 			(font
@@
 			)
 		)
-		(property "Footprint" "inspirefly:IHLP1212BZEZ2R2M1Z"
+		(property "Footprint" "inspirefly:IND_SRP4020FA-2R2M_BRN"
 			(at 422.656 326.136 90)
 			(hide yes)
