File: BatteryHeater/FlatpitchedCable.kicad_pcb (KiCad board)
At the start: 2 copper layers, 45 x 45 mm, 1 part

Commit message: Finalize board work + BOM work
Other:
- board size 45 x 45 mm -> 39.8 x 31.5 mm
