File: FlightController/FlightController.kicad_pcb (KiCad board)
At the start: 4 copper layers, 40 x 40 mm, 39 parts, among them IC1 MX25L25645GM2I-08G-TR, J3 M55-7104042R, J5 Conn_01x02_Pin, SW1 SW_TL1015AF160QG, SW2 SW_TL1015AF160QG, U1 STM32L496RGT6TR, U5 BNO086, U9 TCAN332DCNR, Y2 XTAL_ABS07-32.768KHZ-T, Y3 XTAL_ABS07-32.768KHZ-T

Commit message: Flight Controller V0.2, mech integration
Parts:
- removed J5: Conn_01x02_Pin, Connector_PinHeader_2.54mm:PinHeader_1x02_P2.54mm_Vertical
- moved H5 2.83 mm to (73.6, 35.0)
- moved H6 2.83 mm to (110.6, 35.0)
Routing:
- net GND: vias 23 -> 24
Other:
- board size 40 x 40 mm -> 43 x 43 mm
- board text added: "Flight Controller PQ V0.2"
- board text removed: "Flight Controller PQ V0.1"
